File: Byte4066.kicad_sch (KiCad schematic)
At the start: 6 parts, among them J1 Conn_01x10, J2 Conn_02x08_Odd_Even, U1 4066, U2 4066

Commit message: V1
Parts:
- added J3: Conn_01x10, pads:1x10 pads, symbol Connector_Generic:Conn_01x10
- RN1, RN2: renamed from RN?; footprint (none) -> Resistor_SMD:R_Array_Convex_4x0603
Connections:
- net GND: now also J3.1 (Pin_1)
- net P0: now also J3.2 (Pin_2)
- net P1: now also J3.3 (Pin_3)
- net P2: now also U2.5, J3.4 (Pin_4)
- net P3: now also U2.13, J3.5 (Pin_5)
- net P4: now also U1.6, J3.6 (Pin_6)
- net P5: now also U1.12, J3.7 (Pin_7)
- net P6: now also U1.5, J3.8 (Pin_8)
- net P7: now also U1.13, J3.9 (Pin_9)
- net VCC: now also J3.10 (Pin_10)
- net 5B: now reaches U1.10
- net 5B: now also J2.6 (Pin_6)
- net 5A: now reaches U1.11
- net 5A: now also J2.5 (Pin_5)
- net 4B: now reaches U1.8
- net 4B: now also J2.8 (Pin_8)
- net 4A: now reaches U1.9
- net 4A: now also J2.7 (Pin_7)
- net 2A: now reaches U2.3
- net 2A: now also J2.11 (Pin_11)
- net 2B: now reaches U2.4
- net 2B: now also J2.12 (Pin_12)
- net 7A: now reaches J2.1 (Pin_1)
- net 7A: now also U1.1
- net 3B: now reaches J2.10 (Pin_10)
- net 3B: now also U2.2
- net 7B: now reaches J2.2 (Pin_2)
- net 7B: now also U1.2
- net 6A: now reaches J2.3 (Pin_3)
- net 6A: now also U1.3
- net 6B: now reaches J2.4 (Pin_4)
- net 6B: now also U1.4
- net 3A: now reaches J2.9 (Pin_9)
- net 3A: now also U2.1
